Commit message: add panels-mode world and auto-select world/anchor from ray_mode
Adds ouster_demo_panels.sdf (the rendering counterpart of ouster_demo.sdf:
loads gz-sim-sensors-system/ogre2 instead of gz-sim-altimeter-system) so
ray_mode:=panels has a working world to run in.

The three example launches now switch worlds automatically based on ray_mode:
  raycast (default) → ouster_demo.sdf / turtlebot3_ouster_headless.sdf
  panels            → ouster_demo_panels.sdf

The ouster_standalone and sensor_stack URDFs now derive anchor_type from
ray_mode (altimeter for raycast, camera for panels), mirroring the existing
turtlebot3_ouster.urdf.xacro pattern. The separate anchor_type launch arg is
removed from ouster_standalone.launch.py and sensor_stack.launch.py — a single
ray_mode knob now controls both world selection and anchor type.

Co-Authored-By: Claude Opus 4.8 (1M context) <noreply@anthropic.com>
Claude-Session: https://claude.ai/code/session_017y2HZcbfCtksQF81ymKaT1

File: examples/urdf/ouster_standalone.urdf.xacro (robot description, xacro)
@@ -12,5 +12,7 @@
   <xacro:arg name="metadata_lidar0" default="metadata/os1_64_rev7.json"/>
   <xacro:arg name="ray_mode"       default="raycast"/>
-  <xacro:arg name="anchor_type"    default="altimeter"/>
+  <xacro:property name="ray_mode" value="$(arg ray_mode)"/>
+  <xacro:property name="anchor_type"
+    value="${'altimeter' if ray_mode == 'raycast' else 'camera'}"/>
   <xacro:include filename="$(find gz_sensors_ouster)/examples/urdf/ouster_macro.xacro"/>
   <!-- Root frame -->
@@ -46,5 +48,5 @@
     lidar_hz="10.0"
     enable_imu="true" imu_hz="100.0"
-    ray_mode="$(arg ray_mode)"
-    anchor_type="$(arg anchor_type)"/>
+    ray_mode="${ray_mode}"
+    anchor_type="${anchor_type}"/>
 </robot>

File: examples/urdf/sensor_stack.urdf.xacro (robot description, xacro)
@@ -14,5 +14,7 @@
   <xacro:arg name="metadata_rear"  default="metadata/os0_128_rev7.json"/>
   <xacro:arg name="ray_mode"       default="raycast"/>
-  <xacro:arg name="anchor_type"    default="altimeter"/>
+  <xacro:property name="ray_mode" value="$(arg ray_mode)"/>
+  <xacro:property name="anchor_type"
+    value="${'altimeter' if ray_mode == 'raycast' else 'camera'}"/>
   <xacro:include filename="$(find gz_sensors_ouster)/examples/urdf/ouster_macro.xacro"/>
   <xacro:property name="pi" value="3.14159265359"/>
@@ -48,6 +50,6 @@
     lidar_hz="10.0"
     enable_imu="true" imu_hz="100.0"
-    ray_mode="$(arg ray_mode)"
-    anchor_type="$(arg anchor_type)"/>
+    ray_mode="${ray_mode}"
+    anchor_type="${anchor_type}"/>
   <!-- Rear OS0-128 (short-range, no IMU), looking backward -->
   <xacro:ouster_sensor
@@ -58,5 +60,5 @@
     lidar_hz="10.0"
     enable_imu="false"
-    ray_mode="$(arg ray_mode)"
-    anchor_type="$(arg anchor_type)"/>
+    ray_mode="${ray_mode}"
+    anchor_type="${anchor_type}"/>
 </robot>

File: examples/urdf/turtlebot3_ouster.urdf.xacro (robot description, xacro)
@@ -16,5 +16,5 @@
   an ECM-mirrored scene, so NO render engine / GPU is needed — the headless smoke
   runs anywhere. (Pass ray_mode:=panels for the GpuRays path, which needs a
-  rendering world such as ouster_demo.sdf.)
+  rendering world such as ouster_demo_panels.sdf.)
   Spawn via examples/launch/turtlebot3_ouster.launch.py, which passes an ABSOLUTE
   metadata path (relative paths resolve against an on-disk SDF dir, which does not
